File: RL78Display.kicad_pcb (KiCad board)
At the start: 2 copper layers, 25.8 x 29.5 mm, 29 parts, among them J1 USB_B_Mini, J2 breadboardController, J3 TFT_ATM0130B3, Q1 Q_NMOS_GSD, SW1 SW_Push, SW2 SW_Push, U1 NJM2884U1, U2 RL78G13_64pin, Y1 32.768kHz

Commit message: 基板 V1.1
Parts:
- added R10: 1k, RL78Display:1608Metric, F.Cu at (-10.4, 7.10)
- added R11: 1k, RL78Display:1608Metric, F.Cu at (-11.9, 7.10)
- added R7: 1k, RL78Display:1608Metric, F.Cu at (-5.90, 7.10)
- added R8: 1k, RL78Display:1608Metric, F.Cu at (-7.40, 7.10)
- added R9: 1k, RL78Display:1608Metric, F.Cu at (-8.90, 7.10)
- R2: value 100 -> R
- moved C5 14.2 mm to (6.60, 7.10), turned to 90 degrees
- moved R3 11.9 mm to (3.10, -3.70), turned to 90 degrees
- moved C3 1.40 mm to (-6.00, -3.70)
- moved U1 1.40 mm to (-2.20, -3.50)
- moved C4 1.40 mm to (1.60, -3.70)
- moved C1 0.60 mm to (-10.6, 0.50)
- moved Y1 0.60 mm to (-9.00, 1.60)
- moved C2 0.60 mm to (-10.6, 2.70)
- moved Q1 0.40 mm to (9.10, 7.10)
Connections:
- C5 pad 2: +3V3 -> +5V
- C6 pad 1: +3V3 -> +5V
- J2 pad 7: +3V3 -> +5V
- R1 pad 1: +3V3 -> +5V
- R2 pad 1: +3V3 -> +5V
- U2 pad 15: +3V3 -> +5V
- U2 pad 16: +3V3 -> +5V
Routing:
- net +3V3: track 50.2 -> 24.3 mm, vias 2 -> 0
- net SW_D: track 5.78 -> 26.8 mm
- net +5V: track 54.4 -> 68.7 mm, vias 0 -> 2
- net SW_C: track 10.0 -> 23.3 mm
- net TFT_RESET: track 10.9 -> 23.4 mm
- net GND: track 154.0 -> 166.2 mm, vias 1 -> 3
- net BUZZER: track 17.8 -> 29.8 mm
- net TFT_SDA: track 10.6 -> 21.5 mm
- net TFT_SCL: track 10.7 -> 21.2 mm
- net TFT_CS: track 9.07 -> 18.3 mm
- net TFT_DC: track 8.11 -> 16.8 mm
- net Net-(J3-Pad3): track 9.91 -> 3.26 mm
- net TOOL0: track 16.2 -> 22.1 mm
- net POS_V: track 8.67 -> 14.1 mm, vias 1 -> 0
- net SW_B: track 15.2 -> 11.5 mm
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Other:
- board text added: "RL78 Display V1.1"
- board text removed: "RL78 Display V1.0"

Commit message: 基板 V2.0
Parts:
- removed SW1, SW2: SW_Push, RL78Display:SW_THBP07-043C
- added C10: 0.1uF, RL78Display:1608Metric, F.Cu at (1.65, 13.4)
- added C11: 0.1uF, RL78Display:1608Metric, F.Cu at (-11.6, 11.0)
- added C12: 0.1uF, RL78Display:1608Metric, F.Cu at (-6.75, 13.4)
- added C8: 0.22F, RL78Display:DCK-3R3E224-E, F.Cu at (9.05, 11.5)
- added C9: 0.1uF, RL78Display:1608Metric, F.Cu at (3.15, 13.4)
- added D2: SW_L, RL78Display:1608Metric, F.Cu at (-10.7, -13.2)
- added D3: SW_R, RL78Display:1608Metric, F.Cu at (10.7, -13.2)
- added J4: USB_B_Micro, RL78Display:ZX62-B-5PA, B.Cu at (0.00, -12.6)
- added R12: 1k, RL78Display:1608Metric, F.Cu at (4.65, 13.4)
- added R13: R, RL78Display:1608Metric, F.Cu at (-10.7, -11.8)
- added R14: R, RL78Display:1608Metric, F.Cu at (10.7, -11.8)
- added U3: TTP223, RL78Display:SOT-23-6, F.Cu at (-7.00, -12.5)
- added U4: TTP223, RL78Display:SOT-23-6, F.Cu at (7.00, -12.5)
- added U5: RX8900CE, RL78Display:RX8900CE, F.Cu at (-1.80, 13.3)
- added U6: NJM2864, RL78Display:SOT-23-5, F.Cu at (-9.75, 13.4)
- C5: value 0.1uF -> 1uF
- J1: footprint RL78Display:Mini_Micro_USB_Connector -> RL78Display:UX60SC-MB-5ST
- moved C5 13.4 mm to (-5.25, 13.4), turned to 270 degrees
- moved Q1 3.30 mm to (5.80, 6.95), turned to 180 degrees
- moved C1 0.70 mm to (-11.3, 0.50)
- moved C2 0.70 mm to (-11.3, 2.70)
- moved Y1 0.70 mm to (-9.70, 1.60)
- moved J2 0.65 mm to (8.89, 10.1)
- moved TP1 0.50 mm to (12.0, 1.00)
- moved TP2 0.50 mm to (12.0, 3.00)
- moved TP3 0.50 mm to (12.0, 5.00)
- moved D1 0.25 mm to (-11.9, -8.75)
- moved F1 0.25 mm to (-7.40, -8.75)
- moved L1 0.25 mm to (-8.90, -8.75)
- moved R2 0.25 mm to (-10.4, -8.75)
Connections:
- C5 pad 2: +5V -> +3V0
- TP3 pad 1: LED_Status -> GPIO
- U2 pad 17: (no net) -> RTC_SCL
- U2 pad 18: (no net) -> RTC_SDA
- U2 pad 30: SW_R -> (no net)
- U2 pad 31: SW_L -> (no net)
- U2 pad 32: (no net) -> GPIO
- U2 pad 33: (no net) -> SW_L
- U2 pad 34: (no net) -> SW_R
- U2 pad 35: (no net) -> SW_A
- U2 pad 36: (no net) -> SW_B
- U2 pad 37: (no net) -> SW_C
- U2 pad 38: (no net) -> SW_D
- U2 pad 59: SW_D -> UART1_RX
- U2 pad 60: SW_C -> UART1_TX
- U2 pad 61: SW_B -> (no net)
- U2 pad 62: SW_A -> (no net)
Routing:
- net GND: track 166.2 -> 205.1 mm
- net RTC_SCL: track 0.00 -> 34.9 mm, vias 0 -> 1
- net RTC_SDA: track 0.00 -> 33.7 mm, vias 0 -> 1
- net +5V: track 68.7 -> 98.6 mm
- net SW_L: track 14.2 -> 43.1 mm, vias 0 -> 1
- net UART1_RX: track 0.00 -> 25.5 mm, vias 0 -> 2
- net UART1_TX: track 0.00 -> 23.7 mm, vias 0 -> 2
- net LED_Status: track 34.5 -> 11.4 mm
- net GPIO: track 0.00 -> 17.1 mm
- net +3V0: track 0.00 -> 14.7 mm, vias 0 -> 2
- net Net-(C9-Pad1): track 0.00 -> 13.2 mm
- net SW_D: track 26.8 -> 16.5 mm
- net POS_H: track 14.2 -> 4.21 mm
- net Net-(C8-Pad1): track 0.00 -> 9.34 mm
- net SW_C: track 23.3 -> 15.4 mm
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- added copper zone on B.Cu, net Net-(U3-Pad3)
- added copper zone on B.Cu, net Net-(U4-Pad3)
- removed copper zone on B.Cu, net GND
- removed copper zone on F.Cu, net GND
Other:
- board size 25.8 x 29.5 mm -> 26.8 x 30 mm
- board text added: "GPIO"
- board text added: "RL78 Display V2.0"
- board text removed: "RL78 Display V1.1"
- board text removed: "TP"

Commit message: 基板 V2.1
Parts:
- removed C10, C6: 0.1uF, RL78Display:1608Metric
- added R15: 2k, RL78Display:1608Metric, F.Cu at (-8.90, -2.90)
- added R16: 2k, RL78Display:1608Metric, F.Cu at (-7.40, -2.90)
- moved C2 2.61 mm to (-8.70, 2.90), turned to 180 degrees
- moved C1 2.43 mm to (-10.9, 2.90), turned to 0 degrees
- moved C11 2.38 mm to (-11.9, 13.3), turned to 270 degrees
- moved C7 1.70 mm to (-11.9, -2.90)
- moved R1 1.70 mm to (-10.4, -2.90)
- moved C12 1.45 mm to (-5.30, 13.3)
- moved C5 1.45 mm to (-3.80, 13.3), turned to 90 degrees
- moved U5 1.31 mm to (-0.50, 13.2)
- moved U6 1.15 mm to (-8.60, 13.4)
- moved D1 1.00 mm to (-11.9, -7.75)
- moved F1 1.00 mm to (-7.40, -7.75)
- moved L1 1.00 mm to (-8.90, -7.75)
- moved R2 1.00 mm to (-10.4, -7.75)
- moved R10 0.95 mm to (-10.4, 6.15)
- moved R11 0.95 mm to (-11.9, 6.15)
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Routing:
- net GND: track 205.1 -> 186.3 mm, vias 3 -> 2
- net BUZZER: track 26.3 -> 18.5 mm, vias 3 -> 1
- net +5V: track 98.6 -> 91.7 mm, vias 2 -> 1
- net UART1_TX: track 23.7 -> 30.5 mm
- net SW_L: track 43.1 -> 38.1 mm
- net RTC_SDA: track 33.7 -> 29.0 mm, vias 1 -> 2
- net TOOL0: track 20.7 -> 25.0 mm
- net NRST: track 21.6 -> 25.2 mm, vias 1 -> 2
- net Net-(C9-Pad1): track 13.2 -> 9.87 mm, vias 0 -> 2
- net Net-(F1-Pad2): track 13.8 -> 16.8 mm, vias 2 -> 1
- net RTC_SCL: track 34.9 -> 32.1 mm, vias 1 -> 3
- net UART1_RX: track 25.5 -> 27.8 mm
- net Net-(C7-Pad1): track 4.16 -> 6.16 mm
- net XT1: track 5.00 -> 6.43 mm
- net GPIO: track 17.1 -> 18.3 mm
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Other:
- board text added: "RL78 Display V2.1"
- board text removed: "RL78 Display V2.0"
