File: RL78Display.sch (KiCad schematic (older format))
At the start: 29 parts, among them J1 USB_B_Mini, J2 breadboardController, J3 TFT_ATM0130B3, Q1 Q_NMOS_GSD, SW1 SW_Push, SW2 SW_Push, U1 NJM2884U1, U2 RL78G13_64pin, Y1 32.768kHz

Commit message: 基板 V1.1
Parts:
- added R10, R11, R7, R8, R9: 1k, RL78Display:1608Metric, symbol Device:R_Small
- R2: value 100 -> R
Connections:
- net +3V3: now also R10.2, R11.2, R7.2, R8.2, R9.2; no longer C5.2, C6.1, J2.7 (VDD), R1.1, R2.1, U2.15 (Vdd), U2.16 (EVddo)
- net +5V: now also C5.2, C6.1, J2.7 (VDD), R1.1, R2.1, U2.15 (Vdd), U2.16 (EVddo)
- net TFT_CS: now also R8.1
- net TFT_DC: now also R7.1
- net TFT_RESET: now also R11.1
- net TFT_SCL: now also R9.1
- net TFT_SDA: now also R10.1
Changed lines of the file:
@@
 Sheet 1 1
 Title "RL78Display"
-Date "2021-04-10"
-Rev "V1.0"
+Date "2021-05-07"
+Rev "V1.1"
 Comp "https://github.com/KimiakiK"
 Comment1 ""
@@
 $EndComp
 $Comp
-L power:+3.3V #PWR012
-U 1 1 60741CCD
-P 2150 4750
-F 0 "#PWR012" H 2150 4600 50  0001 C CNN
-F 1 "+3.3V" H 2150 4900 50  0000 C CNN
-F 2 "" H 2150 4750 50  0001 C CNN
-F 3 "" H 2150 4750 50  0001 C CNN
-	1    2150 4750
-	1    0    0    -1
-$EndComp
-$Comp
 L power:GND #PWR09
 U 1 1 6074252E
@@
 Wire Wire Line
 	2150 4750 1750 4750
-Connection ~ 2150 4750
 Text GLabel 1800 1450 2    50   Input ~ 0
 TOOL0
@@
 	1    0    0    -1
 $EndComp
-$Comp
-L power:+3.3V #PWR07
-U 1 1 60746954
-P 3750 2600
-F 0 "#PWR07" H 3750 2450 50  0001 C CNN
-F 1 "+3.3V" H 3750 2750 50  0000 C CNN
-F 2 "" H 3750 2600 50  0001 C CNN
-F 3 "" H 3750 2600 50  0001 C CNN
-	1    3750 2600
-	1    0    0    -1
-$EndComp
 Wire Wire Line
 	3650 2800 3750 2800
@@
 F 3 "~" H 3650 3800 50  0001 C CNN
 	1    3650 3800
-	1    0    0    -1
-$EndComp
-$Comp
-L power:+3.3V #PWR010
-U 1 1 6074B06F
-P 3650 3700
-F 0 "#PWR010" H 3650 3550 50  0001 C CNN
-F 1 "+3.3V" H 3650 3850 50  0000 C CNN
-F 2 "" H 3650 3700 50  0001 C CNN
-F 3 "" H 3650 3700 50  0001 C CNN
-	1    3650 3700
 	1    0    0    -1
 $EndComp
@@
 Text GLabel 4150 5400 0    50   Input ~ 0
 SW_R
-Text GLabel 9100 2950 0    50   Input ~ 0
+Text GLabel 8350 2950 0    50   Input ~ 0
 TFT_DC
-Text GLabel 9100 3050 0    50   Input ~ 0
+Text GLabel 8350 3050 0    50   Input ~ 0
 TFT_CS
-Text GLabel 9100 3150 0    50   Input ~ 0
+Text GLabel 8350 3150 0    50   Input ~ 0
 TFT_SCL
-Text GLabel 9100 3250 0    50   Input ~ 0
+Text GLabel 8350 3250 0    50   Input ~ 0
 TFT_SDA
-Text GLabel 9100 3350 0    50   Input ~ 0
+Text GLabel 8350 3350 0    50   Input ~ 0
 TFT_RESET
 $Comp
@@
 Text GLabel 9000 2450 0    50   Input ~ 0
 TFT_LEDK
-Wire Wire Line
-	9100 2950 9300 2950
-Wire Wire Line
-	9300 3050 9100 3050
-Wire Wire Line
-	9100 3150 9300 3150
-Wire Wire Line
-	9300 3250 9100 3250
-Wire Wire Line
-	9100 3350 9300 3350
 $Comp
 L Device:R_Small R3
@@
 P 9700 1500
 F 0 "R2" V 9600 1500 50  0000 C CNN
-F 1 "100" V 9700 1500 40  0001 C CNN
+F 1 "R" V 9700 1500 40  0001 C CNN
 F 2 "RL78Display:1608Metric" H 9700 1500 50  0001 C CNN
 F 3 "~" H 9700 1500 50  0001 C CNN
 	1    9700 1500
 	0    1    1    0
-$EndComp
-$Comp
-L power:+3.3V #PWR016
-U 1 1 6079A29F
-P 9900 1400
-F 0 "#PWR016" H 9900 1250 50  0001 C CNN
-F 1 "+3.3V" H 9900 1550 50  0000 C CNN
-F 2 "" H 9900 1400 50  0001 C CNN
-F 3 "" H 9900 1400 50  0001 C CNN
-	1    9900 1400
-	1    0    0    -1
 $EndComp
 Wire Wire Line
@@
 	4150 3700 3650 3700
 Connection ~ 4150 3700
-Connection ~ 3650 3700
 Wire Wire Line
 	4150 3600 3900 3600
@@
 Wire Wire Line
 	4150 3400 3200 3400
+$Comp
+L power:+5V #PWR0101
+U 1 1 6094E039
+P 3750 2600
+F 0 "#PWR0101" H 3750 2450 50  0001 C CNN
+F 1 "+5V" H 3750 2750 50  0000 C CNN
+F 2 "" H 3750 2600 50  0001 C CNN
+F 3 "" H 3750 2600 50  0001 C CNN
+	1    3750 2600
+	1    0    0    -1
+$EndComp
+$Comp
+L power:+5V #PWR0102
+U 1 1 609507B9
+P 3650 3700
+F 0 "#PWR0102" H 3650 3550 50  0001 C CNN
+F 1 "+5V" H 3650 3850 50  0000 C CNN
+F 2 "" H 3650 3700 50  0001 C CNN
+F 3 "" H 3650 3700 50  0001 C CNN
+	1    3650 3700
+	1    0    0    -1
+$EndComp
+Connection ~ 3650 3700
+$Comp
+L power:+5V #PWR0103
+U 1 1 609542BE
+P 2150 4750
+F 0 "#PWR0103" H 2150 4600 50  0001 C CNN
+F 1 "+5V" H 2150 4900 50  0000 C CNN
+F 2 "" H 2150 4750 50  0001 C CNN
+F 3 "" H 2150 4750 50  0001 C CNN
+	1    2150 4750
+	1    0    0    -1
+$EndComp
+Connection ~ 2150 4750
+$Comp
+L power:+5V #PWR0104
+U 1 1 60956797
+P 9900 1400
+F 0 "#PWR0104" H 9900 1250 50  0001 C CNN
+F 1 "+5V" H 9900 1550 50  0000 C CNN
+F 2 "" H 9900 1400 50  0001 C CNN
+F 3 "" H 9900 1400 50  0001 C CNN
+	1    9900 1400
+	1    0    0    -1
+$EndComp
+$Comp
+L Device:R_Small R8
+U 1 1 60957FFD
+P 8550 2800
+F 0 "R8" V 8560 2730 50  0000 R TNN
+F 1 "1k" V 8550 2800 40  0000 C CNN
+F 2 "RL78Display:1608Metric" H 8550 2800 50  0001 C CNN
+F 3 "~" H 8550 2800 50  0001 C CNN
+	1    8550 2800
+	-1   0    0    1
+$EndComp
+$Comp
+L Device:R_Small R9
+U 1 1 6095B48D
+P 8650 2800
+F 0 "R9" V 8660 2730 50  0000 R TNN
+F 1 "1k" V 8650 2800 40  0000 C CNN
+F 2 "RL78Display:1608Metric" H 8650 2800 50  0001 C CNN
+F 3 "~" H 8650 2800 50  0001 C CNN
+	1    8650 2800
+	-1   0    0    1
+$EndComp
+$Comp
+L Device:R_Small R10
+U 1 1 6095BBBB
+P 8750 2800
+F 0 "R10" V 8760 2730 50  0000 R TNN
+F 1 "1k" V 8750 2800 40  0000 C CNN
+F 2 "RL78Display:1608Metric" H 8750 2800 50  0001 C CNN
+F 3 "~" H 8750 2800 50  0001 C CNN
+	1    8750 2800
+	-1   0    0    1
+$EndComp
+$Comp
+L Device:R_Small R11
+U 1 1 6095BEEC
+P 8850 2800
+F 0 "R11" V 8860 2730 50  0000 R TNN
+F 1 "1k" V 8850 2800 40  0000 C CNN
+F 2 "RL78Display:1608Metric" H 8850 2800 50  0001 C CNN
+F 3 "~" H 8850 2800 50  0001 C CNN
+	1    8850 2800
+	-1   0    0    1
+$EndComp
+$Comp
+L Device:R_Small R7
+U 1 1 6095C152
+P 8450 2800
+F 0 "R7" V 8460 2730 50  0000 R TNN
+F 1 "1k" V 8450 2800 40  0000 C CNN
+F 2 "RL78Display:1608Metric" H 8450 2800 50  0001 C CNN
+F 3 "~" H 8450 2800 50  0001 C CNN
+	1    8450 2800
+	-1   0    0    1
+$EndComp
+$Comp
+L power:+3.3V #PWR0105
+U 1 1 6095C93B
+P 8450 2550
+F 0 "#PWR0105" H 8450 2400 50  0001 C CNN
+F 1 "+3.3V" H 8450 2700 50  0000 C CNN
+F 2 "" H 8450 2550 50  0001 C CNN
+F 3 "" H 8450 2550 50  0001 C CNN
+	1    8450 2550
+	1    0    0    -1
+$EndComp
+Wire Wire Line
+	8450 2550 8550 2550
+Connection ~ 8450 2550
+Connection ~ 8750 2550
+Wire Wire Line
+	8750 2550 8850 2550
+Connection ~ 8650 2550
+Wire Wire Line
+	8650 2550 8750 2550
+Connection ~ 8550 2550
+Wire Wire Line
+	8550 2550 8650 2550
+Wire Wire Line
+	8350 2950 8450 2950
+Wire Wire Line
+	8350 3050 8550 3050
+Wire Wire Line
+	8350 3150 8650 3150
+Wire Wire Line
+	8350 3250 8750 3250
+Wire Wire Line
+	8450 2900 8450 2950
+Connection ~ 8450 2950
+Wire Wire Line
+	8450 2950 9300 2950
+Wire Wire Line
+	8550 2900 8550 3050
+Connection ~ 8550 3050
+Wire Wire Line
+	8550 3050 9300 3050
+Wire Wire Line
+	8650 2900 8650 3150
+Connection ~ 8650 3150
+Wire Wire Line
+	8650 3150 9300 3150
+Wire Wire Line
+	8750 2900 8750 3250
+Connection ~ 8750 3250
+Wire Wire Line
+	8750 3250 9300 3250
+Wire Wire Line
+	8850 2900 8850 3350
+Connection ~ 8850 3350
+Wire Wire Line
+	8850 3350 8350 3350
+Wire Wire Line
+	8850 3350 9300 3350
+Wire Wire Line
+	8850 2550 8850 2700
+Wire Wire Line
+	8750 2550 8750 2700
+Wire Wire Line
+	8650 2550 8650 2700
+Wire Wire Line
+	8550 2550 8550 2700
+Wire Wire Line
+	8450 2550 8450 2700
 $EndSCHEMATC

Commit message: 基板 V2.0
Parts:
- removed SW1, SW2: SW_Push, RL78Display:SW_THBP07-043C, symbol Switch:SW_Push
- added C10, C11, C12, C9: 0.1uF, RL78Display:1608Metric, symbol Device:C_Small
- added C8: 0.22F, RL78Display:DCK-3R3E224-E, symbol Device:CP_Small
- added D2: SW_L, RL78Display:1608Metric, symbol Device:LED_Small
- added D3: SW_R, RL78Display:1608Metric, symbol Device:LED_Small
- added J4: USB_B_Micro, RL78Display:ZX62-B-5PA, symbol Connector:USB_B_Micro
- added R12: 1k, RL78Display:1608Metric, symbol Device:R_Small
- added R13, R14: R, RL78Display:1608Metric, symbol Device:R_Small
- added U3, U4: TTP223, RL78Display:SOT-23-6, symbol RL78Display:TTP223
- added U5: RX8900CE, RL78Display:RX8900CE, symbol RL78Display:RX8900CE
- added U6: NJM2864, RL78Display:SOT-23-5, symbol RL78Display:NJM2864
- C5: value 0.1uF -> 1uF
- J1: footprint RL78Display:Mini_Micro_USB_Connector -> RL78Display:UX60SC-MB-5ST
Connections:
- net +5V: now also C11.1, U3.5 (VDD), U4.5 (VDD), U6.1 (VIN), U6.3 (CTRL); no longer C5.2
- net GND: now also C10.1, C11.2, C12.2, C8.2, C9.2, D2.1 (K), D3.1 (K), J4.5 (GND), J4.6 (Shield), U3.2 (VSS), U4.2 (VSS), U5.1 (FOE), U5.4 (FOUT), U5.9 (GND), U6.2 (GND)
- net LED_Status: no longer TP3.1
- net SW_A: now also U2.35 (P52); no longer U2.62 (P00/TI00)
- net SW_B: now also U2.36 (P53); no longer U2.61 (P01/TO00)
- net SW_C: now also U2.37 (P54); no longer U2.60 (P02/ANI17/SO10/TxD1)
- net SW_D: now also U2.38 (P55); no longer U2.59 (P03/ANI16/SI10/RxD1/SDA10)
- net SW_L: now also U2.33 (P50/INTP1/SI11/SDA11), R13.2, U3.1 (Q); no longer U2.31 (P05/TI05/TO05)
- net SW_R: now also U2.34 (P51/INTP2/SO11), R14.2, U4.1 (Q); no longer U2.30 (P06/TI06/TO06)
- net at F1.2, J1.1 (VBUS): now also J4.1 (VBUS)
- net RTC_SCL: now reaches U2.17 (P60/SCLA0)
- net RTC_SCL: now also U5.5 (SCL)
- net RTC_SDA: now reaches U2.18 (P61/SDAA0)
- net RTC_SDA: now also U5.7 (SDA)
- net GPIO: now reaches U2.32 (P30/INTP3/RTC1HZ)
- net GPIO: now also TP3.1
- new net: C9.1, R12.1, U5.3 (VBAT)
- new net: C8.1, R12.2
- new net: C12.1, U6.4 (NB)
- new net: D2.2 (A), R13.1
- new net: D3.2 (A), R14.1
- new net +3V0: C10.2, C5.2, U5.2 (VDD), U6.5 (VOUT)
- new net UART1_RX: J4.2 (D-), U2.59 (P03/ANI16/SI10/RxD1/SDA10)
- new net UART1_TX: J4.3 (D+), U2.60 (P02/ANI17/SO10/TxD1)
- no-connect marks 40 -> 43
Other:
- moved on the sheet: C5, D1, J2, R2, TP3

Commit message: 基板 V2.1
Parts:
- removed C10, C6: 0.1uF, RL78Display:1608Metric, symbol Device:C_Small
- added R15, R16: 2k, RL78Display:1608Metric, symbol Device:R_Small
Connections:
- net +5V: now also R15.1, R16.1
- net RTC_SCL: now also R15.2
- net RTC_SDA: now also R16.2
Changed lines of the file:
@@
 Sheet 1 1
 Title "RL78Display"
-Date "2021-06-20"
-Rev "V2.0"
+Date "2021-07-10"
+Rev "V2.1"
 Comp "https://github.com/KimiakiK"
 Comment1 ""
@@
 XT2
 $Comp
-L Device:C_Small C6
-U 1 1 60749CCD
-P 3650 3800
-F 0 "C6" H 3550 3850 50  0000 R CNN
-F 1 "0.1uF" H 3550 3750 50  0000 R CNN
-F 2 "RL78Display:1608Metric" H 3650 3800 50  0001 C CNN
-F 3 "~" H 3650 3800 50  0001 C CNN
-	1    3650 3800
-	1    0    0    -1
-$EndComp
-$Comp
 L power:GND #PWR011
 U 1 1 6074BB14
-P 3650 3900
-F 0 "#PWR011" H 3650 3650 50  0001 C CNN
-F 1 "GND" H 3650 3750 50  0000 C CNN
-F 2 "" H 3650 3900 50  0001 C CNN
-F 3 "" H 3650 3900 50  0001 C CNN
-	1    3650 3900
+P 4050 3800
+F 0 "#PWR011" H 4050 3550 50  0001 C CNN
+F 1 "GND" H 4050 3650 50  0000 C CNN
+F 2 "" H 4050 3800 50  0001 C CNN
+F 3 "" H 4050 3800 50  0001 C CNN
+	1    4050 3800
 	1    0    0    -1
 $EndComp
@@
 Wire Wire Line
 	4150 3600 4150 3500
-Wire Wire Line
-	3900 3600 3900 3900
-Wire Wire Line
-	3900 3900 3650 3900
-Connection ~ 3650 3900
 $Comp
 L power:+5V #PWR0101
@@
 L power:+5V #PWR0102
 U 1 1 609507B9
-P 3650 3700
-F 0 "#PWR0102" H 3650 3550 50  0001 C CNN
-F 1 "+5V" H 3650 3850 50  0000 C CNN
-F 2 "" H 3650 3700 50  0001 C CNN
-F 3 "" H 3650 3700 50  0001 C CNN
-	1    3650 3700
-	1    0    0    -1
-$EndComp
-Connection ~ 3650 3700
+P 3700 3700
+F 0 "#PWR0102" H 3700 3550 50  0001 C CNN
+F 1 "+5V" H 3700 3850 50  0000 C CNN
+F 2 "" H 3700 3700 50  0001 C CNN
+F 3 "" H 3700 3700 50  0001 C CNN
+	1    3700 3700
+	1    0    0    -1
+$EndComp
 $Comp
 L power:+5V #PWR0103
@@
 Text GLabel 6850 2800 2    50   Input ~ 0
 UART1_RX
-Text GLabel 4150 4100 0    50   Input ~ 0
+Text GLabel 3650 4100 0    50   Input ~ 0
 RTC_SCL
-Text GLabel 4150 4200 0    50   Input ~ 0
+Text GLabel 3650 4200 0    50   Input ~ 0
 RTC_SDA
-Connection ~ 4150 3600
 Connection ~ 4150 3700
 Wire Wire Line
-	4150 3700 3650 3700
-Wire Wire Line
-	4150 3600 3900 3600
+	4150 3700 3850 3700
 Wire Wire Line
 	4150 3400 3200 3400
@@
 	1000 7250 1200 7250
 Connection ~ 1200 7250
-$Comp
-L Device:C_Small C10
-U 1 1 60D58FD4
-P 1400 6750
-F 0 "C10" V 1450 6600 50  0000 L CNN
-F 1 "0.1uF" V 1350 6600 50  0000 C CNN
-F 2 "RL78Display:1608Metric" H 1400 6750 50  0001 C CNN
-F 3 "~" H 1400 6750 50  0001 C CNN
-	1    1400 6750
-	0    -1   -1   0
-$EndComp
-Wire Wire Line
-	1300 6650 1300 6750
-Connection ~ 1300 6750
-Wire Wire Line
-	1300 6750 1300 6950
-Wire Wire Line
-	1650 6750 1500 6750
-Connection ~ 1650 6750
 Wire Wire Line
 	1750 6950 1300 6950
@@
 	9100 1250 9400 1250
 Connection ~ 7050 1150
+Wire Wire Line
+	3650 4100 3700 4100
+Wire Wire Line
+	4150 4200 3850 4200
+Wire Wire Line
+	4150 3600 4050 3600
+Wire Wire Line
+	4050 3600 4050 3800
+Connection ~ 4150 3600
+$Comp
+L Device:R_Small R15
+U 1 1 611F3124
+P 3700 3900
+F 0 "R15" V 3750 3900 50  0000 C TNN
+F 1 "2k" V 3700 3900 40  0000 C CNN
+F 2 "RL78Display:1608Metric" H 3700 3900 50  0001 C CNN
+F 3 "~" H 3700 3900 50  0001 C CNN
+	1    3700 3900
+	1    0    0    -1
+$EndComp
+$Comp
+L Device:R_Small R16
+U 1 1 611F5E02
+P 3850 3900
+F 0 "R16" V 3900 3900 50  0000 C TNN
+F 1 "2k" V 3850 3900 40  0000 C CNN
+F 2 "RL78Display:1608Metric" H 3850 3900 50  0001 C CNN
+F 3 "~" H 3850 3900 50  0001 C CNN
+	1    3850 3900
+	1    0    0    -1
+$EndComp
+Connection ~ 3700 3700
+Wire Wire Line
+	3700 3700 3650 3700
+Wire Wire Line
+	3700 4000 3700 4100
+Connection ~ 3700 4100
+Wire Wire Line
+	3700 4100 4150 4100
+Wire Wire Line
+	3700 3800 3700 3700
+Wire Wire Line
+	3850 3700 3850 3800
+Connection ~ 3850 3700
+Wire Wire Line
+	3850 3700 3700 3700
+Wire Wire Line
+	3850 4000 3850 4200
+Connection ~ 3850 4200
+Wire Wire Line
+	3850 4200 3650 4200
+Wire Wire Line
+	1300 6650 1300 6950
 $EndSCHEMATC
